File: 16seg/led_array.kicad_sch (KiCad schematic)
At the start: 18 parts

Commit message: 2023/05/26
Parts:
- added J1 (x2), J7: VCC, Connector_Wire:SolderWire-0.5sqmm_1x01_D0.9mm_OD2.1mm, symbol Connector_Generic:Conn_01x01
- added J10, J4 (x2): CLR, Connector_Wire:SolderWire-0.5sqmm_1x01_D0.9mm_OD2.1mm, symbol Connector_Generic:Conn_01x01
- added J11, J5 (x2): CK, Connector_Wire:SolderWire-0.5sqmm_1x01_D0.9mm_OD2.1mm, symbol Connector_Generic:Conn_01x01
- added J12, J6 (x2): GND, Connector_Wire:SolderWire-0.5sqmm_1x01_D0.9mm_OD2.1mm, symbol Connector_Generic:Conn_01x01
- added J13: A1, Connector_Wire:SolderWire-0.5sqmm_1x01_D0.9mm_OD2.1mm, symbol Connector_Generic:Conn_01x01
- added J14: A2, Connector_Wire:SolderWire-0.5sqmm_1x01_D0.9mm_OD2.1mm, symbol Connector_Generic:Conn_01x01
- added J15: B, Connector_Wire:SolderWire-0.5sqmm_1x01_D0.9mm_OD2.1mm, symbol Connector_Generic:Conn_01x01
- added J16: C, Connector_Wire:SolderWire-0.5sqmm_1x01_D0.9mm_OD2.1mm, symbol Connector_Generic:Conn_01x01
- added J17: D1, Connector_Wire:SolderWire-0.5sqmm_1x01_D0.9mm_OD2.1mm, symbol Connector_Generic:Conn_01x01
- added J18: D2, Connector_Wire:SolderWire-0.5sqmm_1x01_D0.9mm_OD2.1mm, symbol Connector_Generic:Conn_01x01
- added J19: E, Connector_Wire:SolderWire-0.5sqmm_1x01_D0.9mm_OD2.1mm, symbol Connector_Generic:Conn_01x01
- added J2 (x2): deta, Connector_Wire:SolderWire-0.5sqmm_1x01_D0.9mm_OD2.1mm, symbol Connector_Generic:Conn_01x01
- added J20: F, Connector_Wire:SolderWire-0.5sqmm_1x01_D0.9mm_OD2.1mm, symbol Connector_Generic:Conn_01x01
- added J21: G1, Connector_Wire:SolderWire-0.5sqmm_1x01_D0.9mm_OD2.1mm, symbol Connector_Generic:Conn_01x01
- added J22: G2, Connector_Wire:SolderWire-0.5sqmm_1x01_D0.9mm_OD2.1mm, symbol Connector_Generic:Conn_01x01
- added J23: H, Connector_Wire:SolderWire-0.5sqmm_1x01_D0.9mm_OD2.1mm, symbol Connector_Generic:Conn_01x01
- added J24: I, Connector_Wire:SolderWire-0.5sqmm_1x01_D0.9mm_OD2.1mm, symbol Connector_Generic:Conn_01x01
- added J25: J, Connector_Wire:SolderWire-0.5sqmm_1x01_D0.9mm_OD2.1mm, symbol Connector_Generic:Conn_01x01
- added J26: K, Connector_Wire:SolderWire-0.5sqmm_1x01_D0.9mm_OD2.1mm, symbol Connector_Generic:Conn_01x01
- added J27: L, Connector_Wire:SolderWire-0.5sqmm_1x01_D0.9mm_OD2.1mm, symbol Connector_Generic:Conn_01x01
- added J28: M, Connector_Wire:SolderWire-0.5sqmm_1x01_D0.9mm_OD2.1mm, symbol Connector_Generic:Conn_01x01
- added J29, J8: DP, Connector_Wire:SolderWire-0.5sqmm_1x01_D0.9mm_OD2.1mm, symbol Connector_Generic:Conn_01x01
- added J3 (x2), J9: OF, Connector_Wire:SolderWire-0.5sqmm_1x01_D0.9mm_OD2.1mm, symbol Connector_Generic:Conn_01x01
- added Q1, Q10, Q11, Q12, Q13, Q14, Q15, Q16, Q17, Q2, Q3, Q4, Q5, Q6, Q7, Q8, Q9: BSS138, Package_TO_SOT_SMD:SOT-23, symbol Device:Q_NMOS_GSD
- D1: renamed from D2; footprint SOD3716X135N -> Diode_SMD:D_SOD-123
- D10: renamed from D11; footprint SOD3716X135N -> Diode_SMD:D_SOD-123
- D11: renamed from D12; footprint SOD3716X135N -> Diode_SMD:D_SOD-123
- D12: renamed from D13; footprint SOD3716X135N -> Diode_SMD:D_SOD-123
- D13: renamed from D14; footprint SOD3716X135N -> Diode_SMD:D_SOD-123
- D14: renamed from D15; footprint SOD3716X135N -> Diode_SMD:D_SOD-123
- D15: renamed from D16; footprint SOD3716X135N -> Diode_SMD:D_SOD-123
- D16: renamed from D17; footprint SOD3716X135N -> Diode_SMD:D_SOD-123
- D17: renamed from D18; footprint SOD3716X135N -> Diode_SMD:D_SOD-123
- D2: renamed from D3; footprint SOD3716X135N -> Diode_SMD:D_SOD-123
- D3: renamed from D4; footprint SOD3716X135N -> Diode_SMD:D_SOD-123
- D4: renamed from D5; footprint SOD3716X135N -> Diode_SMD:D_SOD-123
- D5: renamed from D6; footprint SOD3716X135N -> Diode_SMD:D_SOD-123
- D6: renamed from D7; footprint SOD3716X135N -> Diode_SMD:D_SOD-123
- D7: renamed from D8; footprint SOD3716X135N -> Diode_SMD:D_SOD-123
- D8: renamed from D9; footprint SOD3716X135N -> Diode_SMD:D_SOD-123
- D9: renamed from D10; footprint SOD3716X135N -> Diode_SMD:D_SOD-123
- seg1: renamed from D1; footprint (none) -> Library:16seg
Connections:
- net at D1.1: now also Q1.3 (D)
- net at D7.1: now also Q7.3 (D)
- net at D11.1: now also Q11.3 (D)
- net at D2.1: now also Q2.3 (D)
- net at D5.1: now also Q5.3 (D)
- net at D16.1: now also Q16.3 (D)
- net at D10.1: now also Q10.3 (D)
- net at D15.1: now also Q15.3 (D)
- net at D12.1: now also Q12.3 (D)
- net at D6.1: now also Q6.3 (D)
- net at D8.1: now also Q8.3 (D)
- net at D13.1: now also Q13.3 (D)
- net at D9.1: now also Q9.3 (D)
- net at D17.1: now also Q17.3 (D)
- net at D4.1: now also Q4.3 (D)
- net at D14.1: now also Q14.3 (D)
- net at D3.1: now also Q3.3 (D)
- net +5V renamed +5F
- net +5F: now also J1.1 (Pin_1), J1.1 (Pin_1), J7.1 (Pin_1)
- new net: J28.1 (Pin_1), Q16.1 (G)
- new net: J19.1 (Pin_1), Q7.1 (G)
- new net: J26.1 (Pin_1), Q14.1 (G)
- new net: J24.1 (Pin_1), Q12.1 (G)
- new net: J14.1 (Pin_1), Q2.1 (G)
- new net: J22.1 (Pin_1), Q10.1 (G)
- new net: J27.1 (Pin_1), Q15.1 (G)
- new net: J23.1 (Pin_1), Q11.1 (G)
- new net: J18.1 (Pin_1), Q6.1 (G)
- new net: J20.1 (Pin_1), Q8.1 (G)
- new net: J16.1 (Pin_1), Q4.1 (G)
- new net: J13.1 (Pin_1), Q1.1 (G)
- new net: J29.1 (Pin_1), Q17.1 (G)
- new net: J25.1 (Pin_1), Q13.1 (G)
- new net: J21.1 (Pin_1), Q9.1 (G)
- new net: J15.1 (Pin_1), Q3.1 (G)
- new net: J17.1 (Pin_1), Q5.1 (G)
- new net CK_LED: J11.1 (Pin_1), J5.1 (Pin_1), J5.1 (Pin_1)
- new net CLR_LED: J10.1 (Pin_1), J4.1 (Pin_1), J4.1 (Pin_1)
- new net DP_LED: J8.1 (Pin_1)
- new net GND2: J12.1 (Pin_1), J6.1 (Pin_1), J6.1 (Pin_1), Q1.2 (S), Q10.2 (S), Q11.2 (S), Q12.2 (S), Q13.2 (S), Q14.2 (S), Q15.2 (S), Q16.2 (S), Q17.2 (S), Q2.2 (S), Q3.2 (S), Q4.2 (S), Q5.2 (S), Q6.2 (S), Q7.2 (S), Q8.2 (S), Q9.2 (S)
- new net OF_LED: J3.1 (Pin_1), J3.1 (Pin_1), J9.1 (Pin_1)
- new net deta_LED: J2.1 (Pin_1), J2.1 (Pin_1)
Other:
- moved on the sheet: D1, D10, D11, D12, D13, D14, D15, D16, D17, D2, D3, D4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
