File: 16seg/16seg.kicad_sch (KiCad schematic)
At the start: 99 parts, among them J1 Conn_01x01, J10 Conn_01x01, J11 Conn_01x01, J12 Conn_01x01, J13 A1, J14 A2, J15 B, J16 C, J17 D1, J18 D2, J19 E, J2 Conn_01x01, J20 F, J21 G1, J22 G2, J23 H, J24 I, J25 J, J26 K, J27 L, J28 M, J29 DP, J3 Conn_01x01, J30 OF, J4 Conn_01x01, J5 Conn_01x01, J6 Conn_01x01, J7 Conn_01x01, J8 Conn_01x01, J9 Conn_01x01

Commit message: 2023/05/27
Parts:
- added R35, R36, R37, R38, R39, R40, R41, R42, R43, R44, R45, R46, R47, R48, R49, R50, R51: 10k, Resistor_SMD:R_1206_3216Metric, symbol Device:R
Connections:
- net GND: now also R35.1, R36.1, R37.1, R38.1, R39.1, R40.1, R41.1, R42.1, R43.1, R44.1, R45.1, R46.1, R47.1, R48.1, R49.1, R50.1, R51.1
- net Q_D: now also R43.2
- net at J25.1 (Pin_1), U13.5 (Q), U14.2 (D): now also R47.2
- net at J23.1 (Pin_1), U11.5 (Q), U12.2 (D): now also R45.2
- net at J14.1 (Pin_1), U2.5 (Q), U3.2 (D): now also R36.2
- net at J15.1 (Pin_1), U3.5 (Q), U4.2 (D): now also R37.2
- net at J16.1 (Pin_1), U4.5 (Q), U5.2 (D): now also R38.2
- net at J22.1 (Pin_1), U10.5 (Q), U11.2 (D): now also R44.2
- net at J18.1 (Pin_1), U6.5 (Q), U7.2 (D): now also R40.2
- net at J19.1 (Pin_1), U7.5 (Q), U8.2 (D): now also R41.2
- net at J28.1 (Pin_1), U16.5 (Q), U17.2 (D): now also R50.2
- net at J13.1 (Pin_1), U1.5 (Q), U2.2 (D): now also R35.2
- net at J17.1 (Pin_1), U5.5 (Q), U6.2 (D): now also R39.2
- net at J20.1 (Pin_1), U8.5 (Q), U9.2 (D): now also R42.2
- net at J29.1 (Pin_1), JP1.1 (A), U17.5 (Q): now also R51.2
- net at J26.1 (Pin_1), U14.5 (Q), U15.2 (D): now also R48.2
- net at J27.1 (Pin_1), U15.5 (Q), U16.2 (D): now also R49.2
- net at J24.1 (Pin_1), U12.5 (Q), U13.2 (D): now also R46.2
Other:
- moved on the sheet: J13, J14, J15, J16, J17, J18, J19, J20, J21, J22, J23, J24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
